Commit message: add cpu case and battery

File: urdf/battery.xacro (robot description, xacro)
@@ -6,5 +6,5 @@
         <origin xyz="0 -1.03 -.45" rpy="0 0 0"/>
         <geometry>
-          <mesh filename="package://vrx_gazebo/models/battery/mesh/battery.dae"/>
+          <mesh filename="package://wamv_description/models/battery/mesh/battery.dae"/>
         </geometry>
       </visual>

File: urdf/cpu_cases.xacro (robot description, xacro)
@@ -6,5 +6,5 @@
       <origin xyz="0.073 0 -1.53" rpy="0 0 0"/>
       <geometry>
-        <mesh filename="package://vrx_gazebo/models/cpu_cases/mesh/cpu_cases.dae"/>
+        <mesh filename="package://wamv_description/models/cpu_cases/mesh/cpu_cases.dae"/>
       </geometry>
     </visual>

File: urdf/wamv_base.urdf.xacro (robot description, xacro)
@@ -1,4 +1,4 @@
 <?xml version="1.0"?>
-<robot xmlns:xacro="http://ros.org/wiki/xacro" name="wam-v">
+<robot xmlns:xacro="http://ros.org/wiki/xacro" name="wam-v-base">
   <!-- Macro for creating the main collisions as simple shapes. -->
   <xacro:macro name="main_collisions" params="prefix reflect:=1">
