Commit message: add dinamixel

File: urdf/wamv.ros2_control.xacro (robot description, xacro)
@@ -1,3 +1,25 @@
 <robot xmlns:xacro="http://ros.org/wiki/xacro" name="engine">
+    <xacro:macro name="engine_propeller_control" params="left_joint right_joint enable_dummy">
+        <ros2_control name="engine_propeller_control" type="system">
+            <hardware>
+                <plugin>dynamixel_hardware_interface/DynamixelHardwareInterface</plugin>
+                <param name="port_name">/dev/ttyUSB0</param>
+                <param name="baudrate">9600</param>
+                <param name="enable_dummy">${enable_dummy}</param>
+            </hardware>
+            <joint name="${left_joint}">
+                <param name="id">1</param>
+                <param name="motor_type">XW540-T260</param>
+                <command_interface name="position"/>
+                <state_interface name="position"/>
+            </joint>
+            <joint name="${right_joint}">
+                <param name="id">2</param>
+                <param name="motor_type">XW540-T260</param>
+                <command_interface name="position"/>
+                <state_interface name="position"/>
+            </joint>
+        </ros2_control>
+    </xacro:macro>
     <xacro:macro name="engine_control" params="ip_address port left_thruster_joint right_thruster_joint enable_dummy">
         <ros2_control name="engine_control" type="system">

File: urdf/wamv.urdf.xacro (robot description, xacro)
@@ -15,7 +15,11 @@
     port="12345"
     enable_dummy="true"
-    left_thruster_joint="left_engine_propeller_joint"
-    right_thruster_joint="right_engine_propeller_joint"
+    left_thruster_joint="left_chasis_engine_joint"
+    right_thruster_joint="right_chasis_engine_joint"
   />
+  <xacro:engine_propeller_control
+    left_joint="left_engine_propeller_joint"
+    right_joint="right_engine_propeller_joint"
+    enable_dummy="true"/>
   <xacro:include filename="$(find wamv_description)/urdf/sensors/lidar.xacro"/>
   <xacro:lidar prefix="front" position="1.0 0 1.2" orientation="0 0 0"/>

Commit message: remove dynamixel hardware interface
Signed-off-by: hakuturu583 <ms.kataoka@gmail.com>

File: urdf/wamv.ros2_control.xacro (robot description, xacro)
@@ -1,29 +1,3 @@
 <robot xmlns:xacro="http://ros.org/wiki/xacro" name="engine">
-    <xacro:macro name="engine_propeller_control" params="left_joint right_joint enable_dummy">
-        <ros2_control name="engine_propeller_control" type="system">
-            <hardware>
-                <plugin>dynamixel_hardware_interface/DynamixelHardwareInterface</plugin>
-                <param name="port_name">/dev/ttyUSB0</param>
-                <param name="baudrate">57600</param>
-                <param name="enable_dummy">${enable_dummy}</param>
-            </hardware>
-            <joint name="${left_joint}">
-                <param name="id">1</param>
-                <param name="motor_type">XW540-T260</param>
-                <command_interface name="position" />
-                <state_interface name="position" />
-                <param name="max_joint_limit">3.14</param>
-                <param name="min_joint_limit">-3.14</param>
-            </joint>
-            <joint name="${right_joint}">
-                <param name="id">2</param>
-                <param name="motor_type">XW540-T260</param>
-                <command_interface name="position" />
-                <state_interface name="position" />
-                <param name="max_joint_limit">3.14</param>
-                <param name="min_joint_limit">-3.14</param>
-            </joint>
-        </ros2_control>
-    </xacro:macro>
     <xacro:macro name="engine_control" params="ip_address port left_thruster_joint right_thruster_joint enable_dummy">
         <ros2_control name="engine_control" type="system">
