Commit message: #15 xacroにros_controlを追加

File: urdf/thrusters/engine.xacro (robot description, xacro)
@@ -2,5 +2,5 @@
 <robot xmlns:xacro="http://ros.org/wiki/xacro" name="wam-v-two-engines">
   <!-- Macro for inserting an engine with its propeller. -->
-  <xacro:macro name="engine" params="prefix position:='0 0 0' orientation:='0 0 0'">
+  <xacro:macro name="engine" params="prefix enable_dummy position:='0 0 0' orientation:='0 0 0' ip_address='192.168.10.100' port=12345">
     <link name="${prefix}_engine_link">
       <visual>
@@ -58,4 +58,12 @@
       <dynamics friction="0.05" damping="0.05" />
     </joint>
+    <xacro:include filename="$(find wamv_description)/urdf/wamv.ros2_control.xacro" />
+    <xacro:engine_control
+      ip_address="${ip_address}"
+      port="${port}"
+      enable_dummy="${enable_dummy}"
+      chasis_engine_joint="${prefix}_chasis_engine_joint"
+      engine_propeller_joint="${prefix}_engine_propeller_joint"
+    />
   </xacro:macro>
 </robot>

File: urdf/wamv.ros2_control.xacro (robot description, xacro)
@@ -1,27 +1,5 @@
-<robot xmlns:xacro="http://ros.org/wiki/xacro" name="azimuth_thruster">
-    <xacro:macro name="azimuth_thruster_control" params="left_joint right_joint enable_dummy">
-        <ros2_control name="azimuth_thruster_control" type="system">
-            <hardware>
-                <plugin>dynamixel_hardware_interface/DynamixelHardwareInterface</plugin>
-                <param name="port_name">/dev/ttyUSB0</param>
-                <param name="baudrate">9600</param>
-                <param name="enable_dummy">${enable_dummy}</param>
-            </hardware>
-            <joint name="${left_joint}">
-                <param name="id">1</param>
-                <param name="motor_type">XW540-T260</param>
-                <command_interface name="position" />
-                <state_interface name="position" />
-            </joint>
-            <joint name="${right_joint}">
-                <param name="id">2</param>
-                <param name="motor_type">XW540-T260</param>
-                <command_interface name="position" />
-                <state_interface name="position" />
-            </joint>
-        </ros2_control>
-    </xacro:macro>
-    <xacro:macro name="main_thruster_control" params="ip_address port left_thruster_joint right_thruster_joint enable_dummy">
-        <ros2_control name="main_thruster_control" type="system">
+<robot xmlns:xacro="http://ros.org/wiki/xacro" name="engine">
+    <xacro:macro name="engine_control" params="ip_address port chasis_engine_joint engine_propeller_joint enable_dummy">
+        <ros2_control name="engine_control" type="system">
             <hardware>
                 <plugin>wamv_control/WamVHardware</plugin>
@@ -29,6 +7,6 @@
                 <param name="port">${port}</param>
                 <param name="timeout_seconds">10.0</param>
-                <param name="left_thruster_joint">${left_thruster_joint}</param>
-                <param name="right_thruster_joint">${right_thruster_joint}</param>
+                <param name="chasis_engine_joint">${chasis_engine_joint}</param>
+                <param name="engine_propeller_joint">${engine_propeller_joint}</param>
                 <param name="enable_dummy">${enable_dummy}</param>
             </hardware>

File: urdf/wamv.urdf.xacro (robot description, xacro)
@@ -8,6 +8,6 @@
   <xacro:battery prefix="right" position="0 -1 0.45" orientation="0 0 0"/>
   <xacro:include filename="$(find wamv_description)/urdf/thrusters/engine.xacro" />
-  <xacro:engine prefix="left" position="-2.373776 1.027135 0.318237" />
-  <xacro:engine prefix="right" position="-2.373776 -1.027135 0.318237" />
+  <xacro:engine prefix="left" enable_dummy="true" position="-2.373776 1.027135 0.318237" />
+  <xacro:engine prefix="right" enable_dummy="true" position="-2.373776 -1.027135 0.318237" />
   <xacro:include filename="$(find wamv_description)/urdf/sensors/lidar.xacro"/>
   <xacro:lidar prefix="front" position="1.0 0 1.2" orientation="0 0 0"/>
@@ -22,5 +22,3 @@
   <xacro:camera prefix="left" position="0.0 -0.6 1.2" orientation="0 0.0 -1.570795"/>
   <xacro:camera prefix="right" position="0.0 0.6 1.2" orientation="0 0.0 1.570795"/>
-  <xacro:include filename="$(find wamv_description)/urdf/thrusters/thruster.xacro"/>
-  <xacro:thruster enable_dummy="false" />
 </robot>

Commit message: #15 joint名修正

File: urdf/thrusters/engine.xacro (robot description, xacro)
@@ -2,5 +2,5 @@
 <robot xmlns:xacro="http://ros.org/wiki/xacro" name="wam-v-two-engines">
   <!-- Macro for inserting an engine with its propeller. -->
-  <xacro:macro name="engine" params="prefix enable_dummy position:='0 0 0' orientation:='0 0 0' ip_address='192.168.10.100' port=12345">
+  <xacro:macro name="engine" params="prefix enable_dummy position:='0 0 0' orientation:='0 0 0'">
     <link name="${prefix}_engine_link">
       <visual>
@@ -58,12 +58,4 @@
       <dynamics friction="0.05" damping="0.05" />
     </joint>
-    <xacro:include filename="$(find wamv_description)/urdf/wamv.ros2_control.xacro" />
-    <xacro:engine_control
-      ip_address="${ip_address}"
-      port="${port}"
-      enable_dummy="${enable_dummy}"
-      chasis_engine_joint="${prefix}_chasis_engine_joint"
-      engine_propeller_joint="${prefix}_engine_propeller_joint"
-    />
   </xacro:macro>
 </robot>

File: urdf/wamv.ros2_control.xacro (robot description, xacro)
@@ -1,4 +1,4 @@
 <robot xmlns:xacro="http://ros.org/wiki/xacro" name="engine">
-    <xacro:macro name="engine_control" params="ip_address port chasis_engine_joint engine_propeller_joint enable_dummy">
+    <xacro:macro name="engine_control" params="ip_address port left_thruster_joint right_thruster_joint enable_dummy">
         <ros2_control name="engine_control" type="system">
             <hardware>
@@ -7,6 +7,6 @@
                 <param name="port">${port}</param>
                 <param name="timeout_seconds">10.0</param>
-                <param name="chasis_engine_joint">${chasis_engine_joint}</param>
-                <param name="engine_propeller_joint">${engine_propeller_joint}</param>
+                <param name="left_thruster_joint">${left_thruster_joint}</param>
+                <param name="right_thruster_joint">${right_thruster_joint}</param>
                 <param name="enable_dummy">${enable_dummy}</param>
             </hardware>

File: urdf/wamv.urdf.xacro (robot description, xacro)
@@ -10,4 +10,12 @@
   <xacro:engine prefix="left" enable_dummy="true" position="-2.373776 1.027135 0.318237" />
   <xacro:engine prefix="right" enable_dummy="true" position="-2.373776 -1.027135 0.318237" />
+  <xacro:include filename="$(find wamv_description)/urdf/wamv.ros2_control.xacro" />
+  <xacro:engine_control
+    ip_address="192.168.10.100"
+    port="12345"
+    enable_dummy="true"
+    left_thruster_joint="left_engine_propeller_joint"
+    right_thruster_joint="right_engine_propeller_joint"
+  />
   <xacro:include filename="$(find wamv_description)/urdf/sensors/lidar.xacro"/>
   <xacro:lidar prefix="front" position="1.0 0 1.2" orientation="0 0 0"/>
